File: backfin_wifi/backfin_wifi.sch (EAGLE design)
At the start: 22 parts

Commit message: First cut V0.0
Parts:
- removed ANT1: PLACEHOLDER, texas:SWRA092B
- removed U$3: TXB0106TSSOP16, knowles_custom:TXB0106TSSOP16
- removed U$4: TLV70236SOT23-5, knowles_custom:TLV70236SOT23-5
- added U$6: AT8010-E2R9HAA, custom:AT8010-E2R9HAA
- added U$7: TLV70236SOT23-5, custom:TLV70236SOT23-5
- added U$8: TXB0106TSSOP16, custom:TXB0106TSSOP16
- U$1: device knowles_custom:CC3000MOD -> custom:CC3000MOD
Connections:
- net GND: now also U$7.GND, U$8.GND; no longer U$3.GND, U$4.GND
- net N$14: now also U$8.B4; no longer U$3.B4
- net N$15: now also U$6.FEED; no longer ANT1.ANTENNA
- net N$16: now also U$8.A1; no longer U$3.A1
- net SPI_CLK_HOST: now also U$8.B2; no longer U$3.B2
- net SPI_CS_HOST: now also U$8.B6; no longer U$3.B6
- net SPI_DIN_HOST: now also U$8.B3; no longer U$3.B3
- net SPI_DOUT_HOST: now also U$8.B5; no longer U$3.B5
- net VBAT_SW_EN: now also U$8.B1; no longer U$3.B1
- net VCC: now also U$7.EN, U$7.IN, U$7.OUT, U$8.OE, U$8.VCCA, U$8.VCCB; no longer U$3.OE, U$3.VCCA, U$3.VCCB, U$4.EN, U$4.IN, U$4.OUT
- net WL_SPI_CLK_HOST: now also U$8.A2; no longer U$3.A2
- net WL_SPI_CS_HOST: now also U$8.A6; no longer U$3.A6
- net WL_SPI_DIN_HOST: now also U$8.A3; no longer U$3.A3
- net WL_SPI_DOUT_HOST: now also U$8.A5; no longer U$3.A5
- net WL_SPI_IRQ_HOST: now also U$8.A4; no longer U$3.A4
Changed lines of the file:
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@@
 <part name="SUPPLY29" library="supply2" deviceset="GND" device=""/>
 <part name="SUPPLY30" library="supply2" deviceset="GND" device=""/>
-<part name="ANT1" library="texas" deviceset="SWRA092B" device="" value="PLACEHOLDER"/>
-<part name="U$4" library="knowles_custom" deviceset="TLV70236" device="SOT23-5"/>
-<part name="U$1" library="knowles_custom" deviceset="CC3000MOD" device=""/>
-<part name="U$3" library="knowles_custom" deviceset="TXB0106" device="TSSOP16"/>
+<part name="U$1" library="custom" deviceset="CC3000MOD" device=""/>
+<part name="U$6" library="custom" deviceset="AT8010-E2R9HAA" device=""/>
+<part name="U$7" library="custom" deviceset="TLV70236" device="SOT23-5"/>
+<part name="U$8" library="custom" deviceset="TXB0106" device="TSSOP16"/>
 </parts>
 <sheets>
@@
 <instance part="SUPPLY29" gate="GND" x="-45.72" y="71.12"/>
 <instance part="SUPPLY30" gate="GND" x="-71.12" y="71.12"/>
-<instance part="ANT1" gate="G$1" x="-93.98" y="104.14"/>
-<instance part="U$4" gate="G$1" x="104.14" y="63.5"/>
 <instance part="U$1" gate="G$1" x="7.62" y="17.78"/>
-<instance part="U$3" gate="G$1" x="109.22" y="-58.42"/>
+<instance part="U$6" gate="G$1" x="-99.06" y="96.52"/>
+<instance part="U$7" gate="G$1" x="104.14" y="63.5"/>
+<instance part="U$8" gate="G$1" x="109.22" y="-58.42"/>
 </instances>
 <busses>
@@
 <wire x1="78.74" y1="53.34" x2="88.9" y2="53.34" width="0.1524" layer="91"/>
 <junction x="88.9" y="53.34"/>
-<pinref part="U$4" gate="G$1" pin="GND"/>
+<pinref part="U$7" gate="G$1" pin="GND"/>
 </segment>
 <segment>
@@
 <wire x1="116.84" y1="-60.96" x2="127" y2="-60.96" width="0.1524" layer="91"/>
 <wire x1="127" y1="-60.96" x2="127" y2="-63.5" width="0.1524" layer="91"/>
-<pinref part="U$3" gate="G$1" pin="GND"/>
+<pinref part="U$8" gate="G$1" pin="GND"/>
 </segment>
 <segment>
@@
 <label x="26.67" y="-58.166" size="1.778" layer="95"/>
 <pinref part="U$1" gate="G$1" pin="SPI_CS"/>
-<pinref part="U$3" gate="G$1" pin="A6"/>
+<pinref part="U$8" gate="G$1" pin="A6"/>
 </segment>
 </net>
@@
 <label x="26.67" y="-55.626" size="1.778" layer="95"/>
 <pinref part="U$1" gate="G$1" pin="SPI_DOUT"/>
-<pinref part="U$3" gate="G$1" pin="A5"/>
+<pinref part="U$8" gate="G$1" pin="A5"/>
 </segment>
 </net>
@@
 <label x="26.67" y="-53.086" size="1.778" layer="95"/>
 <pinref part="U$1" gate="G$1" pin="SPI_IRQ"/>
-<pinref part="U$3" gate="G$1" pin="A4"/>
+<pinref part="U$8" gate="G$1" pin="A4"/>
 </segment>
 </net>
@@
 <label x="26.67" y="-50.546" size="1.778" layer="95"/>
 <pinref part="U$1" gate="G$1" pin="SPI_DIN"/>
-<pinref part="U$3" gate="G$1" pin="A3"/>
+<pinref part="U$8" gate="G$1" pin="A3"/>
 </segment>
 </net>
@@
 <label x="26.924" y="-48.006" size="1.778" layer="95"/>
 <pinref part="U$1" gate="G$1" pin="SPI_CLK"/>
-<pinref part="U$3" gate="G$1" pin="A2"/>
+<pinref part="U$8" gate="G$1" pin="A2"/>
 </segment>
 </net>
@@
 <wire x1="81.28" y1="-43.18" x2="86.36" y2="-43.18" width="0.1524" layer="91"/>
 <pinref part="U$1" gate="G$1" pin="VBAT_SW_EN"/>
-<pinref part="U$3" gate="G$1" pin="A1"/>
+<pinref part="U$8" gate="G$1" pin="A1"/>
 </segment>
 </net>
@@
 <wire x1="71.12" y1="-60.96" x2="86.36" y2="-60.96" width="0.1524" layer="91"/>
 <junction x="71.12" y="-45.72"/>
-<pinref part="U$3" gate="G$1" pin="VCCA"/>
-<pinref part="U$3" gate="G$1" pin="OE"/>
+<pinref part="U$8" gate="G$1" pin="VCCA"/>
+<pinref part="U$8" gate="G$1" pin="OE"/>
 </segment>
 <segment>
@@
 <wire x1="124.46" y1="63.5" x2="124.46" y2="66.04" width="0.1524" layer="91"/>
 <junction x="124.46" y="66.04"/>
-<pinref part="U$4" gate="G$1" pin="OUT"/>
+<pinref part="U$7" gate="G$1" pin="OUT"/>
 </segment>
 <segment>
@@
 <wire x1="127" y1="-38.1" x2="127" y2="-45.72" width="0.1524" layer="91"/>
 <wire x1="127" y1="-45.72" x2="116.84" y2="-45.72" width="0.1524" layer="91"/>
-<pinref part="U$3" gate="G$1" pin="VCCB"/>
+<pinref part="U$8" gate="G$1" pin="VCCB"/>
 </segment>
 <segment>
@@
 <wire x1="78.74" y1="66.04" x2="78.74" y2="63.5" width="0.1524" layer="91"/>
 <junction x="78.74" y="66.04"/>
-<pinref part="U$4" gate="G$1" pin="IN"/>
-<pinref part="U$4" gate="G$1" pin="EN"/>
+<pinref part="U$7" gate="G$1" pin="IN"/>
+<pinref part="U$7" gate="G$1" pin="EN"/>
 </segment>
 </net>
@@
 <wire x1="106.68" y1="17.78" x2="132.08" y2="17.78" width="0.1524" layer="91"/>
 <label x="108.204" y="18.034" size="1.778" layer="95"/>
-<pinref part="U$3" gate="G$1" pin="B1"/>
+<pinref part="U$8" gate="G$1" pin="B1"/>
 </segment>
 </net>
@@
 <pinref part="J1" gate="A" pin="3"/>
 <wire x1="182.88" y1="-38.1" x2="195.58" y2="-38.1" width="0.1524" layer="91"/>
-<pinref part="U$3" gate="G$1" pin="B2"/>
+<pinref part="U$8" gate="G$1" pin="B2"/>
 </segment>
 </net>
@@
 <pinref part="J1" gate="A" pin="4"/>
 <wire x1="218.44" y1="-38.1" x2="203.2" y2="-38.1" width="0.1524" layer="91"/>
-<pinref part="U$3" gate="G$1" pin="B3"/>
+<pinref part="U$8" gate="G$1" pin="B3"/>
 </segment>
 </net>
@@
 <wire x1="195.58" y1="-35.56" x2="180.34" y2="-35.56" width="0.1524" layer="91"/>
 <wire x1="180.34" y1="-35.56" x2="180.34" y2="-55.88" width="0.1524" layer="91"/>
-<pinref part="U$3" gate="G$1" pin="B5"/>
+<pinref part="U$8" gate="G$1" pin="B5"/>
 </segment>
 </net>
@@
 <wire x1="106.68" y1="12.7" x2="132.08" y2="12.7" width="0.1524" layer="91"/>
 <label x="108.204" y="12.954" size="1.778" layer="95"/>
-<pinref part="U$3" gate="G$1" pin="B6"/>
+<pinref part="U$8" gate="G$1" pin="B6"/>
 </segment>
 </net>
@@
 <wire x1="116.84" y1="-53.34" x2="160.02" y2="-53.34" width="0.1524" layer="91"/>
 <label x="134.112" y="-53.086" size="1.778" layer="95"/>
-<pinref part="U$3" gate="G$1" pin="B4"/>
+<pinref part="U$8" gate="G$1" pin="B4"/>
 </segment>
 </net>
@@
 <wire x1="-60.96" y1="96.52" x2="-71.12" y2="96.52" width="0.1524" layer="91"/>
 <wire x1="-71.12" y1="96.52" x2="-71.12" y2="91.44" width="0.1524" layer="91"/>
-<pinref part="ANT1" gate="G$1" pin="ANTENNA"/>
-<wire x1="-93.98" y1="99.06" x2="-93.98" y2="96.52" width="0.1524" layer="91"/>
 <wire x1="-93.98" y1="96.52" x2="-71.12" y2="96.52" width="0.1524" layer="91"/>
 <junction x="-71.12" y="96.52"/>
-</segment>
-</net>
+<pinref part="U$6" gate="G$1" pin="FEED"/>
+</segment>
+</net>
